Commit message: afadsf

File: new_urdf_description/urdf/materials.xacro (robot description, xacro)
@@ -1,5 +1,5 @@
 <?xml version="1.0" ?>
 <robot name="new_urdf" xmlns:xacro="http://www.ros.org/wiki/xacro" >
-<material name="silver">
+<material name="new_urdf_silver">
   <color rgba="0.700 0.700 0.700 1.000"/>
 </material>
